File: Hardware_Filter_SSS/Hardware_Filter_SSS.kicad_sch (KiCad schematic)
At the start: 37 parts, among them U1 LM324, U2 LM324

Commit message: updated hardware, cleaned up
Parts:
- RV21: footprint (none) -> Potentiometer_THT:Potentiometer_Bourns_3386P_Vertical
Changed lines of the file:
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@@
       (effects (font (size 1.27 1.27)) (justify right))
     )
-    (property "Footprint" "" (at 72.39 148.59 0)
+    (property "Footprint" "Potentiometer_THT:Potentiometer_Bourns_3386P_Vertical" (at 72.39 148.59 0)
       (effects (font (size 1.27 1.27)) hide)
     )
